File: USB/USB.kicad_sch (KiCad schematic)
At the start: 22 parts, among them J1 USBC-4-0-CX90MW9-24P1, U2 ESDA25L, U3 USB SWITCH 2CHANNEL TS3USB221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, U6 usb-polarity-TUSB321RWBR

Commit message: add GND test point
Parts:
- added J6: (no value), COMATEL THD:COMATEL_385.0358.1.02.400, symbol SPIRIT-components:2-pin-header
Connections:
- net GND: now also J6.1, J6.2
Other:
- note added: "GND TEST POINT"
Changed lines of the file:
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@@
 		)
 	)
+	(text "GND TEST POINT"
+		(exclude_from_sim no)
+		(at 565.912 330.962 0)
+		(effects
+			(font
+				(size 1.27 1.27)
+				(thickness 0.254)
+				(bold yes)
+			)
+		)
+	)
 	(text "reverse CC pins if mux is driven incorrectly\n(this will invert the MUX_POL signal)"
 		(exclude_from_sim no)
@@
 	)
 	(junction
+		(at 558.8 345.44)
+		(diameter 0)
+		(color 0 0 0 0)
+	)
+	(junction
 		(at 322.58 297.18)
 		(diameter 0)
@@
 	(wire
 		(pts
+			(xy 558.8 340.36) (xy 558.8 345.44)
+		)
+		(stroke
+			(width 0)
+			(type default)
+		)
+	)
+	(wire
+		(pts
 			(xy 142.24 114.3) (xy 153.67 114.3)
 		)
@@
 	)
 	(symbol
+		(lib_id "power:GND")
+		(at 558.8 345.44 0)
+		(unit 1)
+		(body_style 1)
+		(exclude_from_sim no)
+		(in_bom yes)
+		(on_board yes)
+		(in_pos_files yes)
+		(dnp no)
+		(property "Reference" "#PWR071"
+			(at 558.8 351.79 0)
+			(hide yes)
+			(show_name no)
+			(do_not_autoplace no)
+			(effects
+				(font
+					(size 1.27 1.27)
+				)
+			)
+		)
+		(property "Value" "GND"
+			(at 558.8 349.25 0)
+			(show_name no)
+			(do_not_autoplace no)
+			(effects
+				(font
+					(size 1.27 1.27)
+				)
+			)
+		)
+		(property "Footprint" ""
+			(at 558.8 345.44 0)
+			(hide yes)
+			(show_name no)
+			(do_not_autoplace no)
+			(effects
+				(font
+					(size 1.27 1.27)
+				)
+			)
+		)
+		(property "Datasheet" ""
+			(at 558.8 345.44 0)
+			(hide yes)
+			(show_name no)
+			(do_not_autoplace no)
+			(effects
+				(font
+					(size 1.27 1.27)
+				)
+			)
+		)
+		(property "Description" ""
+			(at 558.8 345.44 0)
+			(hide yes)
+			(show_name no)
+			(do_not_autoplace no)
+			(effects
+				(font
+					(size 1.27 1.27)
+				)
+			)
+		)
+		(pin "1"
+		)
+		(instances
+			(project "USB"
+				(path "/96ef50de-934d-4dd6-87fd-3fc40e345030"
+					(reference "#PWR071")
+					(unit 1)
+				)
+			)
+		)
+	)
+	(symbol
 		(lib_name "GND_38")
 		(lib_id "power:GND")
@@
 					(unit 1)
 				)
+			)
+		)
+	)
+	(symbol
+		(lib_id "SPIRIT-components:2-pin-header")
+		(at 566.42 342.9 0)
+		(unit 1)
+		(body_style 1)
+		(exclude_from_sim no)
+		(in_bom yes)
+		(on_board yes)
+		(in_pos_files yes)
+		(dnp no)
+		(fields_autoplaced yes)
+		(property "Reference" "J6"
+			(at 572.77 341.6299 0)
+			(show_name no)
+			(do_not_autoplace no)
+			(effects
+				(font
+					(size 1.27 1.27)
+				)
+				(justify left)
+			)
+		)
+		(property "Value" ""
+			(at 572.77 344.1699 0)
+			(show_name no)
+			(do_not_autoplace no)
+			(effects
+				(font
+					(size 1.27 1.27)
+				)
+				(justify left)
+			)
+		)
+		(property "Footprint" "COMATEL THD:COMATEL_385.0358.1.02.400"
+			(at 566.42 335.28 0)
+			(hide yes)
+			(show_name no)
+			(do_not_autoplace no)
+			(effects
+				(font
+					(size 1.27 1.27)
+				)
+			)
+		)
+		(property "Datasheet" ""
+			(at 566.42 335.28 0)
+			(hide yes)
+			(show_name no)
+			(do_not_autoplace no)
+			(effects
+				(font
+					(size 1.27 1.27)
+				)
+			)
+		)
+		(property "Description" ""
+			(at 566.42 335.28 0)
+			(hide yes)
+			(show_name no)
+			(do_not_autoplace no)
+			(effects
+				(font
+					(size 1.27 1.27)
+				)
+			)
+		)
+		(pin "2"
+		)
+		(pin "1"
+		)
+		(instances
+			(project "USB"
+				(path "/96ef50de-934d-4dd6-87fd-3fc40e345030"
+					(reference "J6")
+					(unit 1)
+				)

Commit message: engi 2026-08-13 voicechat review
Connections:
- no-connect marks 33 -> 31
Other:
- note added: "wrong connection double check"
Changed lines of the file:
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@@
+		)
+	)
+	(text ""
+		(exclude_from_sim no)
+		(at 355.6 110.236 0)
+		(effects
+			(font
+				(size 1.27 1.27)
+			)
 		)
 	)
@@
 				(thickness 0.254)
 				(bold yes)
+			)
+		)
+	)
+	(text "wrong connection double check"
+		(exclude_from_sim no)
+		(at 294.64 123.19 0)
+		(effects
+			(font
+				(size 1.27 1.27)
 			)
 		)
@@
 	)
 	(no_connect
-		(at 203.2 53.34)
-	)
-	(no_connect
 		(at 420.37 285.75)
 	)
@@
 	)
 	(no_connect
-		(at 330.2 -78.74)
-	)
-	(no_connect

Commit message: add packaging info, remove bad fields, format BOM for PCBWAY
Parts:
- C5, C6, C7, R2, R3, R4: Package (none) -> 0603
- D1, D2: Check_prices https://www.snapeda.com/parts/TPD1E05U06DPYR/UMW/view-part/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 -> (none); DigiKey_Part_Number 4518-TPD1E05U06DPYRCT-ND -> (none); MANUFACTURER TI -> (none); MF UMW -> (none); MP TPD1E05U06DPYR -> (none); MPN (none) -> TPD1E05U06DPYR; Package None -> X1SON, 2; SnapEDA_Link https://www.snapeda.com/parts/TPD1E05U06DPYR/UMW/view-part/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 -> (none)
- J1: MANUFACTURER Hirose Electric Co Ltd -> (none); MAXIMUM_PACKAGE_HEIGHT 2.525mm -> (none); PARTREV 24.05.01 -> (none); STANDARD Manufacturer Recommendations -> (none)
- J2, J3, J4, J5, J6: now not fitted
- MUX1: MPN (none) -> HD3SS460RHRR; Package (none) -> 28-WQFN (5.5x3.5)
- Module1: Field4 Amphenol -> (none); Field5 2x 10164227-1001A1RLF -> (none); MPN (none) -> 10164227-1001A1RLF
- R1: MANUFACTURER Panasonic -> (none); MAXIMUM_PACKAGE_HEIGHT 0.6 mm -> (none); MPN (none) -> RC0805JR-071KL; PARTREV 3/1/2020 -> (none); Package (none) -> 0805; STANDARD Manufacturer Recommendations -> (none)
- TVS1, TVS2: Availability In Stock -> (none); Check_prices https://www.snapeda.com/parts/EMI8142MUTAG/Onsemi/view-part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 -> (none); Description_1 4 Line Common Mode Choke Surface Mount 100mA DCR 6Ohm (Typ) -> (none); MANUFACTURER On Semiconductor -> (none); MAXIMUM_PACKAGE_HIEGHT 0.5mm -> (none); MF ON Semiconductor -> (none); MPN EMI8142MUTAG -> EMI8142; PARTREV 0 -> (none); Package XDFN-10 ON Semiconductor -> XDFN10; Price None -> (none); STANDARD IPC-7351B -> (none); SnapEDA_Link https://www.snapeda.com/parts/EMI8142MUTAG/Onsemi/view-part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 -> (none)
- TVS3: value (none) -> 2 Line Common Mode Choke with ESD 100mA DCR 6Ohm; Package (none) -> XDFN6
- U2: Package (none) -> SOT-23-3
- U3: Package (none) -> RSE (UQFN, 10)
- U6: MPN (none) -> TUSB321RWBR; Package (none) -> X2QFN (12)
