File: USB-rev-2/USB-rev-2.kicad_pcb (KiCad board)
At the start: 4 copper layers, 70.3 x 60 mm, 26 parts, among them J1 USBC-4-0-CX90MW9-24P1, U2 ESDA25L, U3 USB SWITCH 2CHANNEL TS3USB221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, U6 usb-polarity-TUSB321RWBR

Commit message: more stitching, improve EMI and graphics
Parts:
- added G***: LOGO, LOGO, F.Cu at (115.1, 65.0)
- moved G*** 28.3 mm to (125.2, 104.1)
- moved G*** 8.87 mm to (103.8, 73.7)
- moved J3 2.86 mm to (114.5, 77.6)
- moved J2 2.21 mm to (114.4, 81.4)
Routing:
- net 5V: track 100.0 -> 84.7 mm
- net CC2: track 31.2 -> 28.8 mm
- net CC2-jumpered: track 65.4 -> 64.2 mm
- net CC1-jumpered: track 61.6 -> 60.6 mm
- net CC1: track 19.7 -> 18.8 mm
- net GND: vias 71 -> 111
Other:
- board text added: "TEST CARRIER 1"
- board text removed: "WELCOME TO USB HELL"
